File: PCB/ADS1299-test_circuit.kicad_pcb (KiCad board)
At the start: 2 copper layers, 100.5 x 95.8 mm, 109 parts, among them J1 CONN_01X07, P1 +5V, P10 CONN_01X03, P11 CONN_01X03, P12 CONN_01X03, P13 CONN_01X03, P14 BiasOut_C, P15 BiasOut_R, P16 BiasIn_C, P17 BiasIn_R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

Commit message: Funcionando para consutlas
Other:
- net class Default removed
